Commit message: All Week2 Assinments Complete

File: src/hrwros_week2/urdf/hrwros_assignment1.xacro (robot description, xacro)
@@ -20,4 +20,5 @@
   <xacro:include filename="$(find hrwros_support)/urdf/bin/bin.urdf.xacro"/>
   <xacro:bin_urdf prefix="bin_1_"/>
+  <xacro:bin_urdf prefix="bin_2_"/>
   <!-- Joints -->
   <joint name="world_interface_to_world" type="fixed">
@@ -72,3 +73,9 @@
   </joint>
   <!-- Add your solution to assignment 1 here -->
+  <!-- bin 2 Assignment1 -->
+  <joint name="bin_2_joint" type="fixed">
+    <parent link="world_interface" />
+    <child link="bin_2_base_link" />
+    <origin xyz="2.1 2.0 0" rpy="0 0 0" />
+  </joint>
 </robot>

File: src/hrwros_week2/urdf/hrwros_assignment2.xacro (robot description, xacro)
@@ -72,3 +72,20 @@
   </joint>
   <!-- Add your solution to assignment 2 here -->
+  <!-- green sphere Assignment2 -->
+  <link name="sphere_link">
+    <visual>
+      <origin xyz="0 0 0.4" />
+      <geometry>
+        <sphere radius="0.4" />
+      </geometry>
+      <material name="sphere_color">
+        <color rgba="0 0.5 0 1"/>
+      </material>
+    </visual>
+  </link>
+  <joint name="sphere_joint" type="fixed">
+    <parent link="world" />
+    <child link="sphere_link" />
+    <origin xyz="5.6 -5 0" />
+  </joint>
 </robot>
